Commit message: + updated robot model

File: ros_robot/urdf/ros_robot.xacro (robot description, xacro)
@@ -22,5 +22,5 @@
       <origin xyz="0 0 0" rpy=" 0 0 0"/>
       <geometry>
-        <box size=".4 .2 .1"/>
+        <box size=".8 .3 .2"/>
       </geometry>
     </collision>
@@ -28,9 +28,9 @@
       <origin xyz="0 0 0" rpy=" 0 0 0"/>
       <geometry>
-        <box size=".4 .2 .1"/>
+        <box size=".8 .3 .2"/>
       </geometry>
     </visual>
     <collision name='back_caster_collision'>
-      <origin xyz="-0.15 0 -0.05" rpy=" 0 0 0"/>
+      <origin xyz="-0.30 0 -0.1" rpy=" 0 0 0"/>
       <geometry>
         <sphere radius="0.0499"/>
@@ -38,5 +38,5 @@
     </collision>
     <visual name='back_caster_visual'>
-      <origin xyz="-0.15 0 -0.05" rpy=" 0 0 0"/>
+      <origin xyz="-0.30 0 -0.1" rpy=" 0 0 0"/>
       <geometry>
         <sphere radius="0.05"/>
@@ -44,5 +44,5 @@
     </visual>
     <collision name='front_caster_collision'>
-      <origin xyz="0.15 0 -0.05" rpy=" 0 0 0"/>
+      <origin xyz="0.30 0 -0.1" rpy=" 0 0 0"/>
       <geometry>
         <sphere radius="0.0499"/>
@@ -50,5 +50,5 @@
     </collision>
     <visual name='front_caster_visual'>
-      <origin xyz="0.15 0 -0.05" rpy=" 0 0 0"/>
+      <origin xyz="0.30 0 -0.1" rpy=" 0 0 0"/>
       <geometry>
         <sphere radius="0.05"/>
@@ -57,14 +57,14 @@
   </link>
   <gazebo reference="chassis">
-    <material>Gazebo/Blue</material>
+    <material>Gazebo/Black</material>
   </gazebo>
   <gazebo reference="left_wheel">
-    <material>Gazebo/Green</material>
+    <material>Gazebo/White</material>
   </gazebo>
   <gazebo reference="right_wheel">
-    <material>Gazebo/Green</material>
+    <material>Gazebo/White</material>
   </gazebo>
   <gazebo reference="camera">
-    <material>Gazebo/Red</material>
+    <material>Gazebo/DarkGrey</material>
   </gazebo>
   <link name="left_wheel">
@@ -72,5 +72,5 @@
 	<origin xyz="0 0 0" rpy="0 1.5707 1.5707"/>
 	<geometry>
-	  <cylinder radius="0.1" length="0.05"/>
+	  <cylinder radius="0.15" length="0.1"/>
 	</geometry>
     </visual>
@@ -78,5 +78,5 @@
 	<origin xyz="0 0 0" rpy="0 1.5707 1.5707"/>
 	<geometry>
-	  <cylinder radius="0.1" length="0.05"/>
+	  <cylinder radius="0.15" length="0.1"/>
 	</geometry>
     </collision>
@@ -95,5 +95,5 @@
 	<origin xyz="0 0 0" rpy="0 1.5707 1.5707"/>
 	<geometry>
-	  <cylinder radius="0.1" length="0.05"/>
+	  <cylinder radius="0.15" length="0.1"/>
 	</geometry>
     </visual>
@@ -101,5 +101,5 @@
 	<origin xyz="0 0 0" rpy="0 1.5707 1.5707"/>
 	<geometry>
-	  <cylinder radius="0.1" length="0.05"/>
+	  <cylinder radius="0.15" length="0.1"/>
 	</geometry>
     </collision>
@@ -115,5 +115,5 @@
   </link>
   <joint type="continuous" name="left_wheel_hinge">
-    <origin xyz="0 0.15 0" rpy="0 0 0"/>
+    <origin xyz="0 0.25 0" rpy="0 0 0"/>
     <child link="left_wheel"/>
     <parent link="chassis"/>
@@ -123,5 +123,5 @@
   </joint>
   <joint type="continuous" name="right_wheel_hinge">
-    <origin xyz="0 -0.15 0" rpy="0 0 0"/>
+    <origin xyz="0 -0.25 0" rpy="0 0 0"/>
     <child link="right_wheel"/>
     <parent link="chassis"/>
@@ -156,5 +156,5 @@
   <!-- CAMERA - JOINT -->
   <joint type="fixed" name="camera_joint">
-    <origin xyz="0.2 0 0" rpy="0 0 0"/>
+    <origin xyz="0.4 0 0" rpy="0 0 0"/>
     <child link="camera"/>
     <parent link="chassis"/>
@@ -189,5 +189,5 @@
   <!-- LIDAR - JOINT -->
   <joint type="fixed" name="hokuyo_joint">
-    <origin xyz="0.15 0 0.1" rpy="0 0 0"/>
+    <origin xyz="0.25 0 0.1" rpy="0 0 0"/>
     <child link="hokuyo"/>
     <parent link="chassis"/>
